File: AlignBit/AlignBit.kicad_pcb (KiCad board)
At the start: 2 copper layers, 38 x 38 mm, 10 parts, among them J1 Conn_01x04_Pin, U1 STM32C011J_4-6_Mx, U4 VL53L0CXV0DH_1, U5 VL53L0CXV0DH_1, U6 VL53L0CXV0DH_1, U7 VL53L0CXV0DH_1

Commit message: Adding things untill its done
Parts:
- added C1: GRM033R61A104ME15J, KiCad:CAPC0603X33N, F.Cu at (184.2, 33.0)
- added C11: C0402C271K5RAC, KiCad:CAPC1005X55N, F.Cu at (177.5, 59.7)
- added C12: GRM188R61C106MA73J, KiCad:CAPC1608X90N, F.Cu at (176.7, 56.1)
- added C13: GRM033R61A104ME15J, KiCad:CAPC0603X33N, F.Cu at (176.8, 42.2)
- added C14: GRT155R61A475ME13J, KiCad:CAPC1005X55N, F.Cu at (175.0, 42.2)
- added C2: GRM033R61A104ME15J, KiCad:CAPC0603X33N, F.Cu at (194.9, 54.1)
- added C3: GRM033R61A104ME15J, KiCad:CAPC0603X33N, F.Cu at (183.2, 66.4)
- added C4: GRM033R61A104ME15J, KiCad:CAPC0603X33N, F.Cu at (162.9, 45.9)
- added C5: GRT155R61A475ME13J, KiCad:CAPC1005X55N, F.Cu at (176.0, 34.5)
- added C6: GRT155R61A475ME13J, KiCad:CAPC1005X55N, F.Cu at (195.9, 52.8)
- added C7: GRT155R61A475ME13J, KiCad:CAPC1005X55N, F.Cu at (181.9, 65.6)
- added C8: GRT155R61A475ME13J, KiCad:CAPC1005X55N, F.Cu at (162.1, 47.2)
- added C9: GRM033R61A104ME15J, KiCad:CAPC0603X33N, F.Cu at (185.7, 52.6)
- added Ce: GRM033R61A104ME15J, KiCad:CAPC0603X33N, F.Cu at (181.9, 55.9)
- added L1: SRN2012T-6R8K, KiCad:INDPM2012X120N, F.Cu at (184.4, 54.6)
- added R1: 0603WAJ0103T5E, KiCad:RESC1608X55N, F.Cu at (164.9, 54.9)
Connections:
- U2 pad 1: +12V -> Net-(U2-+Vin)
- U4 pad 5: unconnected-(U4-XSHUT-Pad5) -> Net-(U4-XSHUT)
- U5 pad 5: unconnected-(U5-XSHUT-Pad5) -> Net-(U4-XSHUT)
- U6 pad 5: unconnected-(U6-XSHUT-Pad5) -> Net-(U4-XSHUT)
- U7 pad 5: unconnected-(U7-XSHUT-Pad5) -> Net-(U4-XSHUT)
Routing:
- net Net-(U4-XSHUT): track 0.00 -> 62.2 mm, vias 0 -> 5
- net 3.3V: track 157.1 -> 175.1 mm
- net INTERNAL_GND: track 144.2 -> 154.9 mm
- net SCL: track 101.2 -> 108.9 mm, vias 6 -> 7
- net Net-(U2-+Vin): track 0.00 -> 4.36 mm
- net +12V: track 8.81 -> 5.26 mm
- net GND: track 12.6 -> 15.8 mm
- net Net-(C13-Pad1): track 0.00 -> 0.99 mm
- net SDA: track 122.4 -> 121.9 mm, vias 9 -> 8

Commit message: adding ppt
Routing:
- net SCL: track 108.9 -> 109.2 mm, vias 7 -> 6
Changed lines of the file:
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@@
   (via (at 160.930702 50.038) (size 0.8) (drill 0.4) (layers "F.Cu" "B.Cu") (net 1))
   (via (at 176.022 64.516) (size 0.8) (drill 0.4) (layers "F.Cu" "B.Cu") (net 1))
-  (via (at 185.42 43.18) (size 0.8) (drill 0.4) (layers "F.Cu" "B.Cu") (free) (net 1))
+  (via (at 185.42 43.18) (size 1) (drill 0.5) (layers "F.Cu" "B.Cu") (free) (net 1))
   (via (at 178.562 44.704) (size 0.8) (drill 0.4) (layers "F.Cu" "B.Cu") (net 1))
   (via (at 195.58 50.038) (size 0.8) (drill 0.4) (layers "F.Cu" "B.Cu") (net 1))
   (via (at 181.864 35.052) (size 0.8) (drill 0.4) (layers "F.Cu" "B.Cu") (net 1))
   (via (at 193.4005 52.832) (size 0.8) (drill 0.4) (layers "F.Cu" "B.Cu") (net 1))
-  (via (at 185.42 35.56) (size 0.8) (drill 0.4) (layers "F.Cu" "B.Cu") (free) (net 1))
+  (via (at 185.42 35.56) (size 1) (drill 0.5) (layers "F.Cu" "B.Cu") (free) (net 1))
   (segment (start 163.068 40.386) (end 164.338 39.116) (width 0.25) (layer "B.Cu") (net 1))
   (segment (start 167.386 39.116) (end 167.513 39.243) (width 0.25) (layer "B.Cu") (net 1))
@@
   (segment (start 161.646338 46.149692) (end 161.646338 47.189662) (width 0.25) (layer "F.Cu") (net 2))
   (segment (start 175.225 44.941751) (end 175.225 44.248249) (width 0.25) (layer "F.Cu") (net 2))
-  (via (at 182.88 40.64) (size 0.8) (drill 0.4) (layers "F.Cu" "B.Cu") (free) (net 2))
+  (via (at 182.88 40.64) (size 1) (drill 0.5) (layers "F.Cu" "B.Cu") (free) (net 2))
   (via (at 161.646338 46.149692) (size 0.8) (drill 0.4) (layers "F.Cu" "B.Cu") (free) (net 2))
   (via (at 171.45 62.738) (size 0.8) (drill 0.4) (layers "F.Cu" "B.Cu") (net 2))
@@
   (via (at 173.482 34.798) (size 0.8) (drill 0.4) (layers "F.Cu" "B.Cu") (free) (net 2))
   (via (at 177.292 32.258) (size 0.8) (drill 0.4) (layers "F.Cu" "B.Cu") (free) (net 2))
-  (via (at 182.88 33.02) (size 0.8) (drill 0.4) (layers "F.Cu" "B.Cu") (free) (net 2))
+  (via (at 182.88 33.02) (size 1) (drill 0.5) (layers "F.Cu" "B.Cu") (free) (net 2))
   (segment (start 182.118 66.802) (end 182.118 66.548) (width 0.25) (layer "B.Cu") (net 2))
   (segment (start 164.338 52.832) (end 164.338 55.118) (width 0.25) (layer "B.Cu") (net 2))
@@
   (segment (start 195.5 51.6) (end 195.5 51.1) (width 0.25) (layer "F.Cu") (net 3))
   (segment (start 182.046387 66.071613) (end 182.118 66) (width 0.25) (layer "F.Cu") (net 3))
-  (via (at 185.42 33.02) (size 0.8) (drill 0.4) (layers "F.Cu" "B.Cu") (free) (net 3))
-  (via (at 185.42 40.64) (size 0.8) (drill 0.4) (layers "F.Cu" "B.Cu") (free) (net 3))
+  (via (at 185.42 33.02) (size 1) (drill 0.5) (layers "F.Cu" "B.Cu") (free) (net 3))
+  (via (at 185.42 40.64) (size 1) (drill 0.5) (layers "F.Cu" "B.Cu") (free) (net 3))
   (segment (start 177.5 51) (end 175.314 51) (width 0.25) (layer "B.Cu") (net 3))
   (segment (start 175.19 51.124) (end 175.19 58.1) (width 0.25) (layer "B.Cu") (net 3))
@@
   (segment (start 160.743397 49.2) (end 160.205702 49.737695) (width 0.25) (layer "F.Cu") (net 6))
   (segment (start 161.7 49.2) (end 160.743397 49.2) (width 0.25) (layer "F.Cu") (net 6))
-  (segment (start 182.118 36.068) (end 181.864 36.068) (width 0.25) (layer "F.Cu") (net 6))
   (segment (start 178.308 35.814) (end 178.308 34.908) (width 0.25) (layer "F.Cu") (net 6))
   (segment (start 184.658 44.958) (end 182.88 43.18) (width 0.25) (layer "F.Cu") (net 6))
@@
   (segment (start 197.358 50.8) (end 196.3 50.8) (width 0.25) (layer "F.Cu") (net 6))
   (segment (start 181.475 44.595) (end 181.475 44.585) (width 0.25) (layer "F.Cu") (net 6))
-  (segment (start 182.626 35.56) (end 182.118 36.068) (width 0.25) (layer "F.Cu") (net 6))
   (segment (start 182.181305 51) (end 184.658 48.523305) (width 0.25) (layer "F.Cu") (net 6))
   (segment (start 179.8 65.7) (end 179.8 65.2) (width 0.25) (layer "F.Cu") (net 6))
@@
   (via (at 162.56 55.118) (size 0.8) (drill 0.4) (layers "F.Cu" "B.Cu") (net 6))
   (via (at 162.56 49.784) (size 0.4) (drill 0.2) (layers "F.Cu" "B.Cu") (free) (net 6))
-  (via (at 182.88 35.56) (size 0.8) (drill 0.4) (layers "F.Cu" "B.Cu") (free) (net 6))
-  (via (at 182.88 43.18) (size 0.8) (drill 0.4) (layers "F.Cu" "B.Cu") (free) (net 6))
-  (via (at 181.864 36.068) (size 0.8) (drill 0.4) (layers "F.Cu" "B.Cu") (net 6))
+  (via (at 182.88 35.56) (size 1) (drill 0.5) (layers "F.Cu" "B.Cu") (free) (net 6))
+  (via (at 182.88 43.18) (size 1) (drill 0.5) (layers "F.Cu" "B.Cu") (free) (net 6))
   (via (at 197.358 50.8) (size 0.8) (drill 0.4) (layers "F.Cu" "B.Cu") (net 6))
+  (segment (start 165.354 47.631312) (end 165.354 43.18) (width 0.25) (layer "B.Cu") (net 6))
   (segment (start 176.793305 64.262) (end 176.322305 63.791) (width 0.25) (layer "B.Cu") (net 6))
-  (segment (start 181.864 36.068) (end 172.466 36.068) (width 0.25) (layer "B.Cu") (net 6))
-  (segment (start 164.193037 48.445652) (end 164.193037 49.784) (width 0.25) (layer "B.Cu") (net 6))
+  (segment (start 182.372 36.068) (end 182.88 35.56) (width 0.25) (layer "B.Cu") (net 6))
+  (segment (start 162.56 49.784) (end 164.193037 49.784) (width 0.25) (layer "B.Cu") (net 6))
+  (segment (start 165.354 43.18) (end 172.466 36.068) (width 0.25) (layer "B.Cu") (net 6))
   (segment (start 197.104 53.848) (end 197.104 52.452396) (width 0.25) (layer "B.Cu") (net 6))
-  (segment (start 164.193037 49.784) (end 162.56 49.784) (width 0.25) (layer "B.Cu") (net 6))
   (segment (start 186.69 64.262) (end 197.104 53.848) (width 0.25) (layer "B.Cu") (net 6))
-  (segment (start 172.466 36.068) (end 165.354 43.18) (width 0.25) (layer "B.Cu") (net 6))
+  (segment (start 164.193037 48.445652) (end 165.007377 47.631312) (width 0.25) (layer "B.Cu") (net 6))
   (segment (start 168.735 63.791) (end 168.714 63.812) (width 0.25) (layer "B.Cu") (net 6))
   (segment (start 179.832 64.262) (end 176.793305 64.262) (width 0.25) (layer "B.Cu") (net 6))
-  (segment (start 165.007377 47.631312) (end 164.193037 48.445652) (width 0.25) (layer "B.Cu") (net 6))
   (segment (start 179.832 64.262) (end 179.832 65.024) (width 0.25) (layer "B.Cu") (net 6))
   (segment (start 162.56 56.134) (end 163.068 56.642) (width 0.25) (layer "B.Cu") (net 6))
+  (segment (start 172.466 36.068) (end 182.372 36.068) (width 0.25) (layer "B.Cu") (net 6))
   (segment (start 163.068 56.642) (end 163.068 58.166) (width 0.25) (layer "B.Cu") (net 6))
   (segment (start 179.832 65.024) (end 179.832 65.168) (width 0.25) (layer "B.Cu") (net 6))
@@
   (segment (start 176.322305 63.791) (end 168.735 63.791) (width 0.25) (layer "B.Cu") (net 6))
   (segment (start 179.832 64.262) (end 186.69 64.262) (width 0.25) (layer "B.Cu") (net 6))
+  (segment (start 164.193037 49.784) (end 164.193037 48.445652) (width 0.25) (layer "B.Cu") (net 6))
+  (segment (start 165.007377 47.631312) (end 165.354 47.631312) (width 0.25) (layer "B.Cu") (net 6))
   (segment (start 162.56 55.118) (end 162.56 56.134) (width 0.25) (layer "B.Cu") (net 6))
   (segment (start 163.068 58.166) (end 168.714 63.812) (width 0.25) (layer "B.Cu") (net 6))
-  (segment (start 165.354 47.631312) (end 165.007377 47.631312) (width 0.25) (layer "B.Cu") (net 6))
-  (segment (start 165.354 43.18) (end 165.354 47.631312) (width 0.25) (layer "B.Cu") (net 6))
   (segment (start 197.104 52.452396) (end 197.358 50.8) (width 0.25) (layer "B.Cu") (net 6))
   (segment (start 197.358 50.8) (end 197.104 50.8) (width 0.25) (layer "B.Cu") (net 6))
